File: KiCad/jjy_sim_esp32_c3.kicad_sch (KiCad schematic)
At the start: 61 parts, among them J1 UART, J2 BAT, M1 NEJI_M3, M2 NEJI_M3, M3 NEJI_M3, M4 NEJI_M3, P1 USB_C_Plug_USB2.0, Q1 BSS84, Q2 2PD601AR, Q3 HN1C01FU-GR (1/2)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

Commit message: C3,C4定数変更、C5をR18に変更
Parts:
- removed C5: 0.1u, Capacitor_SMD:C_0603_1608Metric, symbol Device:C
- added R18: 100k, Resistor_SMD:R_0603_1608Metric, symbol Device:R
- C3, C4: value 0.1u -> 1nF
Connections:
- net GND: now also R18.2
- net at Q1.2 (S), R5.2: now also R18.1
Changed lines of the file:
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@@
 			)
 		)
-		(property "Value" "0.1u"
+		(property "Value" "1nF"
 			(at 228.6 156.21 0)
 			(effects
@@
 			)
 		)
-		(property "Value" "0.1u"
+		(property "Value" "1nF"
 			(at 219.71 156.21 0)
 			(effects
@@
 	)
 	(symbol
-		(lib_id "Device:C")
+		(lib_id "Device:R")
 		(at 205.74 153.67 0)
 		(unit 1)
@@
 		(on_board yes)
 		(dnp no)
-		(property "Reference" "C5"
-			(at 207.01 151.13 0)
+		(property "Reference" "R18"
+			(at 208.28 153.67 90)
 			(effects
 				(font
 					(size 1.27 1.27)
 				)
-				(justify left)
 			)
 		)
-		(property "Value" "0.1u"
-			(at 207.01 156.21 0)
+		(property "Value" "100k"
+			(at 205.74 153.67 90)
 			(effects
 				(font
 					(size 1.27 1.27)
 				)
-				(justify left)
 			)
 		)
-		(property "Footprint" "Capacitor_SMD:C_0603_1608Metric"
-			(at 206.7052 157.48 0)
+		(property "Footprint" "Resistor_SMD:R_0603_1608Metric"
+			(at 203.962 153.67 90)
 			(effects
 				(font
@@
 			(project "jjy_sim_esp32_c3"
 				(path "/e25ad002-4691-4057-a0e9-472916ce3092"
-					(reference "C5")
+					(reference "R18")
 					(unit 1)
 				)
